File: PCB/dronebox_pcb.kicad_sch (KiCad schematic)
At the start: 0 parts

Commit message: schem done
Parts:
- added C101, C102: C_Polarized, symbol Device:C_Polarized
- added C103: C, symbol Device:C
- added J101: Conn_02x05_Odd_Even, symbol Connector_Generic:Conn_02x05_Odd_Even
- added J102: Barrel_Jack_Switch, symbol Connector:Barrel_Jack_Switch
- added J103, J104: Conn_01x02_Female, symbol Connector:Conn_01x02_Female
- added R101: 4K7, symbol Device:R
- added R102: 10K, symbol Device:R
- added R103: 10M, symbol Device:R
- added R104: 680K, symbol Device:R
- added R105: 100K, symbol Device:R
- added RV101: 10K TUNE, Potentiometer_THT:Potentiometer_Bourns_3386F_Vertical, symbol Device:R_Potentiometer_Trim
- added RV102: 100K CV, Potentiometer_THT:Potentiometer_Bourns_3386F_Vertical, symbol Device:R_Potentiometer_Trim
- added RV103: 100K TUNE ALL, Potentiometer_THT:Potentiometer_Bourns_3386F_Vertical, symbol Device:R_Potentiometer_Trim
- added RV104: 200K CV STARVE, Potentiometer_THT:Potentiometer_Bourns_3386F_Vertical, symbol Device:R_Potentiometer_Trim
- added U101: LM386, symbol Amplifier_Audio:LM386
Connections:
- new net: C102.2, J103.1 (Pin_1)
- new net: R104.2, RV103.1
- new net: C101.1, U101.8 (GAIN)
- new net: C101.2, U101.1 (GAIN)
- new net: R102.1, U101.5
- new net: C102.1, R102.2, RV101.3
- new net: J104.1 (Pin_1), RV102.1
- new net: R103.1, RV102.2
- new net: C103.1, RV101.1, RV101.2
- new net: R105.1, RV103.3
- new net: R105.2, RV104.3
- new net +12V: J101.10 (Pin_10), J101.9 (Pin_9), J102.2, R104.1, U101.6 (V+)
- new net CV: R103.2, RV103.2
- new net GND: C103.2, J101.3 (Pin_3), J101.4 (Pin_4), J101.5 (Pin_5), J101.6 (Pin_6), J101.7 (Pin_7), J101.8 (Pin_8), J102.1, J103.2 (Pin_2), J104.2 (Pin_2), R101.1, RV102.3, RV104.1, RV104.2, U101.2 (-), U101.4 (GND)
- new net OUT: R101.2, U101.3 (+)
- no-connect marks 0 -> 4
Other:
- added sheet oscillator (oscillator.kicad_sch)
- added sheet oscillator1 (oscillator.kicad_sch)
- added sheet oscillator10 (oscillator.kicad_sch)
- added sheet oscillator11 (oscillator.kicad_sch)
- added sheet oscillator12 (oscillator.kicad_sch)
- added sheet oscillator13 (oscillator.kicad_sch)
- added sheet oscillator14 (oscillator.kicad_sch)
- added sheet oscillator15 (oscillator.kicad_sch)
- added sheet oscillator16 (oscillator.kicad_sch)
- added sheet oscillator17 (oscillator.kicad_sch)
- added sheet oscillator18 (oscillator.kicad_sch)
- added sheet oscillator19 (oscillator.kicad_sch)
- added sheet oscillator2 (oscillator.kicad_sch)
- added sheet oscillator20 (oscillator.kicad_sch)
- added sheet oscillator21 (oscillator.kicad_sch)
- added sheet oscillator22 (oscillator.kicad_sch)
- added sheet oscillator23 (oscillator.kicad_sch)
- added sheet oscillator24 (oscillator.kicad_sch)
- added sheet oscillator25 (oscillator.kicad_sch)
- added sheet oscillator26 (oscillator.kicad_sch)
- added sheet oscillator27 (oscillator.kicad_sch)
- added sheet oscillator28 (oscillator.kicad_sch)
- added sheet oscillator29 (oscillator.kicad_sch)
- added sheet oscillator3 (oscillator.kicad_sch)
- added sheet oscillator30 (oscillator.kicad_sch)
- added sheet oscillator31 (oscillator.kicad_sch)
- added sheet oscillator32 (oscillator.kicad_sch)
- added sheet oscillator33 (oscillator.kicad_sch)
- added sheet oscillator34 (oscillator.kicad_sch)
- added sheet oscillator35 (oscillator.kicad_sch)
- added sheet oscillator36 (oscillator.kicad_sch)
- added sheet oscillator37 (oscillator.kicad_sch)
- added sheet oscillator38 (oscillator.kicad_sch)
- added sheet oscillator39 (oscillator.kicad_sch)
- added sheet oscillator4 (oscillator.kicad_sch)
- added sheet oscillator40 (oscillator.kicad_sch)
- added sheet oscillator41 (oscillator.kicad_sch)
- added sheet oscillator42 (oscillator.kicad_sch)
- added sheet oscillator43 (oscillator.kicad_sch)
- added sheet oscillator44 (oscillator.kicad_sch)
- added sheet oscillator45 (oscillator.kicad_sch)
- added sheet oscillator46 (oscillator.kicad_sch)
- added sheet oscillator47 (oscillator.kicad_sch)
- added sheet oscillator48 (oscillator.kicad_sch)
- added sheet oscillator49 (oscillator.kicad_sch)
- added sheet oscillator5 (oscillator.kicad_sch)
- added sheet oscillator50 (oscillator.kicad_sch)
- added sheet oscillator51 (oscillator.kicad_sch)
- added sheet oscillator52 (oscillator.kicad_sch)
- added sheet oscillator53 (oscillator.kicad_sch)
- added sheet oscillator54 (oscillator.kicad_sch)
- added sheet oscillator55 (oscillator.kicad_sch)
- added sheet oscillator56 (oscillator.kicad_sch)
- added sheet oscillator57 (oscillator.kicad_sch)
- added sheet oscillator58 (oscillator.kicad_sch)
- added sheet oscillator59 (oscillator.kicad_sch)
- added sheet oscillator6 (oscillator.kicad_sch)
- added sheet oscillator60 (oscillator.kicad_sch)
- added sheet oscillator61 (oscillator.kicad_sch)
- added sheet oscillator62 (oscillator.kicad_sch)
- added sheet oscillator63 (oscillator.kicad_sch)
- added sheet oscillator64 (oscillator.kicad_sch)
- added sheet oscillator65 (oscillator.kicad_sch)
- added sheet oscillator66 (oscillator.kicad_sch)
- added sheet oscillator67 (oscillator.kicad_sch)
- added sheet oscillator68 (oscillator.kicad_sch)
- added sheet oscillator69 (oscillator.kicad_sch)
- added sheet oscillator7 (oscillator.kicad_sch)
- added sheet oscillator70 (oscillator.kicad_sch)
- added sheet oscillator71 (oscillator.kicad_sch)
- added sheet oscillator72 (oscillator.kicad_sch)
- added sheet oscillator73 (oscillator.kicad_sch)
- added sheet oscillator74 (oscillator.kicad_sch)
- added sheet oscillator75 (oscillator.kicad_sch)
- added sheet oscillator76 (oscillator.kicad_sch)
- added sheet oscillator77 (oscillator.kicad_sch)
- added sheet oscillator78 (oscillator.kicad_sch)
- added sheet oscillator79 (oscillator.kicad_sch)
- added sheet oscillator8 (oscillator.kicad_sch)
- added sheet oscillator80 (oscillator.kicad_sch)
- added sheet oscillator81 (oscillator.kicad_sch)
- added sheet oscillator82 (oscillator.kicad_sch)
- added sheet oscillator83 (oscillator.kicad_sch)
- added sheet oscillator84 (oscillator.kicad_sch)
- added sheet oscillator85 (oscillator.kicad_sch)
- added sheet oscillator86 (oscillator.kicad_sch)
- added sheet oscillator87 (oscillator.kicad_sch)
- added sheet oscillator88 (oscillator.kicad_sch)
- added sheet oscillator89 (oscillator.kicad_sch)
- added sheet oscillator9 (oscillator.kicad_sch)
- added sheet oscillator90 (oscillator.kicad_sch)
- added sheet oscillator91 (oscillator.kicad_sch)
- added sheet oscillator92 (oscillator.kicad_sch)
- added sheet oscillator93 (oscillator.kicad_sch)
- added sheet oscillator94 (oscillator.kicad_sch)
- added sheet oscillator95 (oscillator.kicad_sch)
- added sheet oscillator96 (oscillator.kicad_sch)
- added sheet oscillator97 (oscillator.kicad_sch)
- added sheet oscillator98 (oscillator.kicad_sch)
- added sheet oscillator99 (oscillator.kicad_sch)
