File: PCB/oscillator.kicad_sch (KiCad schematic)
At the start: 10 parts, among them Q201 OPT FET, Q202 TRANSISTOR

Commit message: assign fps
Parts:
- renumbered C201 to C4201, D201 to D4201, D202 to D4202, Q201 to Q4201, Q202 to Q4202, R201 to R4201, R202 to R4202, R203 to R4203, RV201 to RV4201, RV202 to RV4202
Changed lines of the file:
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@@
   (symbol (lib_id "power:+12V") (at 133.35 62.23 0)
     (in_bom yes) (on_board yes) (fields_autoplaced)
-    (property "Reference" "#PWR010102" (id 0) (at 133.35 66.04 0)
+    (property "Reference" "#PWR04202" (id 0) (at 133.35 66.04 0)
       (effects (font (size 1.27 1.27)) hide)
     )
@@
   (symbol (lib_id "power:GND") (at 130.81 124.46 0)
     (in_bom yes) (on_board yes) (fields_autoplaced)
-    (property "Reference" "#PWR010101" (id 0) (at 130.81 130.81 0)
+    (property "Reference" "#PWR04201" (id 0) (at 130.81 130.81 0)
       (effects (font (size 1.27 1.27)) hide)
     )
@@
   (symbol (lib_id "power:GND") (at 161.29 76.2 0)
     (in_bom yes) (on_board yes) (fields_autoplaced)
-    (property "Reference" "#PWR010103" (id 0) (at 161.29 82.55 0)
+    (property "Reference" "#PWR04203" (id 0) (at 161.29 82.55 0)
       (effects (font (size 1.27 1.27)) hide)
     )
@@
   (symbol (lib_id "power:GND") (at 176.53 100.33 0)
     (in_bom yes) (on_board yes) (fields_autoplaced)
-    (property "Reference" "#PWR010104" (id 0) (at 176.53 106.68 0)
+    (property "Reference" "#PWR04204" (id 0) (at 176.53 106.68 0)
       (effects (font (size 1.27 1.27)) hide)
     )
@@
   (symbol (lib_id "Device:R") (at 143.51 77.47 0)
     (in_bom yes) (on_board yes) (fields_autoplaced)
-    (property "Reference" "R201" (id 0) (at 146.05 76.1999 0)
+    (property "Reference" "R4201" (id 0) (at 146.05 76.1999 0)
       (effects (font (size 1.27 1.27)) (justify left))
     )
@@
   (symbol (lib_id "Device:R") (at 157.48 69.85 90)
     (in_bom yes) (on_board yes) (fields_autoplaced)
-    (property "Reference" "R202" (id 0) (at 157.48 63.5 90))
+    (property "Reference" "R4202" (id 0) (at 157.48 63.5 90))
     (property "Value" "47K" (id 1) (at 157.48 66.04 90))
     (property "Footprint" "Resistor_THT:R_Axial_DIN0207_L6.3mm_D2.5mm_P2.54mm_Vertical" (id 2) (at 157.48 71.628 90)
@@
   (symbol (lib_id "Device:R") (at 167.64 109.22 0)
     (in_bom yes) (on_board yes) (fields_autoplaced)
-    (property "Reference" "R203" (id 0) (at 170.18 107.9499 0)
+    (property "Reference" "R4203" (id 0) (at 170.18 107.9499 0)
       (effects (font (size 1.27 1.27)) (justify left))
     )
@@
   (symbol (lib_id "Device:D") (at 167.64 116.84 90)
     (in_bom yes) (on_board yes) (fields_autoplaced)
-    (property "Reference" "D202" (id 0) (at 170.18 115.5699 90)
+    (property "Reference" "D4202" (id 0) (at 170.18 115.5699 90)
       (effects (font (size 1.27 1.27)) (justify right))
     )
@@
   (symbol (lib_id "Device:LED") (at 143.51 104.14 90)
     (in_bom yes) (on_board yes) (fields_autoplaced)
-    (property "Reference" "D201" (id 0) (at 147.32 103.2508 90)
+    (property "Reference" "D4201" (id 0) (at 147.32 103.2508 90)
       (effects (font (size 1.27 1.27)) (justify right))
     )
@@
   (symbol (lib_id "Device:C_Polarized") (at 118.11 90.17 0)
     (in_bom yes) (on_board yes) (fields_autoplaced)
-    (property "Reference" "C201" (id 0) (at 121.92 88.8999 0)
+    (property "Reference" "C4201" (id 0) (at 121.92 88.8999 0)
       (effects (font (size 1.27 1.27)) (justify left))
     )
@@
   (symbol (lib_id "Device:R_Potentiometer_Trim") (at 143.51 69.85 90) (mirror x)
     (in_bom yes) (on_board yes) (fields_autoplaced)
-    (property "Reference" "RV201" (id 0) (at 143.51 63.5 90))
+    (property "Reference" "RV4201" (id 0) (at 143.51 63.5 90))
     (property "Value" "10K TUNE" (id 1) (at 143.51 66.04 90))
     (property "Footprint" "Potentiometer_THT:Potentiometer_Bourns_3386F_Vertical" (id 2) (at 143.51 69.85 0)
@@
   (symbol (lib_id "Device:R_Potentiometer_Trim") (at 167.64 97.79 90) (mirror x)
     (in_bom yes) (on_board yes) (fields_autoplaced)
-    (property "Reference" "RV202" (id 0) (at 167.64 91.44 90))
+    (property "Reference" "RV4202" (id 0) (at 167.64 91.44 90))
     (property "Value" "100K LVL" (id 1) (at 167.64 93.98 90))
     (property "Footprint" "Potentiometer_THT:Potentiometer_Bourns_3386F_Vertical" (id 2) (at 167.64 97.79 0)
@@
   (symbol (lib_id "Transistor_BJT:2N3904") (at 140.97 90.17 0) (mirror x)
     (in_bom yes) (on_board yes) (fields_autoplaced)
-    (property "Reference" "Q202" (id 0) (at 146.05 88.8999 0)
+    (property "Reference" "Q4202" (id 0) (at 146.05 88.8999 0)
       (effects (font (size 1.27 1.27)) (justify left))
     )
@@
   (symbol (lib_id "Device:Q_NMOS_GDS") (at 128.27 114.3 0) (mirror x)
     (in_bom yes) (on_board yes) (fields_autoplaced)
-    (property "Reference" "Q201" (id 0) (at 134.62 113.0299 0)
-      (effects (font (size 1.27 1.27)) (justify left))
-    )
+    (property "Reference" "Q4201" (id 0) (at 134.62 113.0299 0)
+      (effects (font (size 1.27 1.27)) (justify left))
+    )

Commit message: rough prices
Parts:
- C4201: Price (none) -> 0.05
- D4201: Price (none) -> 0.03
- D4202: Price (none) -> 0.01
- Q4201: Price (none) -> 0.2
- Q4202: Price (none) -> 0.02
- R4201, R4202, R4203: Price (none) -> 0.015
- RV4201, RV4202: Price (none) -> 0.06
Changed lines of the file:
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@@
+      (effects (font (size 1.27 1.27)) hide)
+    )
+    (property "Price" "0.015" (id 4) (at 143.51 77.47 0)
       (effects (font (size 1.27 1.27)) hide)
     )
@@
     )
     (property "Datasheet" "~" (id 3) (at 157.48 69.85 0)
+      (effects (font (size 1.27 1.27)) hide)
+    )
+    (property "Price" "0.015" (id 4) (at 157.48 69.85 0)
       (effects (font (size 1.27 1.27)) hide)
     )
@@
       (effects (font (size 1.27 1.27)) hide)
     )
+    (property "Price" "0.015" (id 4) (at 167.64 109.22 0)
+      (effects (font (size 1.27 1.27)) hide)
+    )
     (pin "1")
     (pin "2")
@@
     )
     (property "Datasheet" "~" (id 3) (at 167.64 116.84 0)
+      (effects (font (size 1.27 1.27)) hide)
+    )
+    (property "Price" "0.01" (id 4) (at 167.64 116.84 0)
       (effects (font (size 1.27 1.27)) hide)
     )
@@
       (effects (font (size 1.27 1.27)) hide)
     )
+    (property "Price" "0.03" (id 4) (at 143.51 104.14 0)
+      (effects (font (size 1.27 1.27)) hide)
+    )
     (pin "1")
     (pin "2")
@@
       (effects (font (size 1.27 1.27)) hide)
     )
+    (property "Price" "0.05" (id 4) (at 118.11 90.17 0)
+      (effects (font (size 1.27 1.27)) hide)
+    )
     (pin "1")
     (pin "2")
@@
     )
     (property "Datasheet" "~" (id 3) (at 143.51 69.85 0)
+      (effects (font (size 1.27 1.27)) hide)
+    )
+    (property "Price" "0.06" (id 4) (at 143.51 69.85 0)
       (effects (font (size 1.27 1.27)) hide)
     )
@@
     )
     (property "Datasheet" "~" (id 3) (at 167.64 97.79 0)
+      (effects (font (size 1.27 1.27)) hide)
+    )
+    (property "Price" "0.06" (id 4) (at 167.64 97.79 0)
       (effects (font (size 1.27 1.27)) hide)
     )
@@
       (effects (font (size 1.27 1.27)) (justify left) hide)
     )
+    (property "Price" "0.02" (id 4) (at 140.97 90.17 0)
+      (effects (font (size 1.27 1.27)) hide)
+    )
     (pin "1")
     (pin "2")
@@
       (effects (font (size 1.27 1.27)) hide)
     )
+    (property "Price" "0.2" (id 4) (at 128.27 114.3 0)
+      (effects (font (size 1.27 1.27)) hide)
+    )

Commit message: update to smd components
Parts:
- Q9602: renamed from Q4202; footprint Package_TO_SOT_THT:TO-92_Inline -> Package_TO_SOT_SMD:SOT-23
- R9601: renamed from R4201; footprint Resistor_THT:R_Axial_DIN0207_L6.3mm_D2.5mm_P2.54mm_Vertical -> Resistor_SMD:R_1206_3216Metric_Pad1.30x1.75mm_HandSolder
- R9602: renamed from R4202; footprint Resistor_THT:R_Axial_DIN0207_L6.3mm_D2.5mm_P2.54mm_Vertical -> Resistor_SMD:R_1206_3216Metric_Pad1.30x1.75mm_HandSolder
- R9603: renamed from R4203; footprint Resistor_THT:R_Axial_DIN0207_L6.3mm_D2.5mm_P2.54mm_Vertical -> Resistor_SMD:R_1206_3216Metric_Pad1.30x1.75mm_HandSolder
- renumbered C4201 to C9601, D4201 to D9601, D4202 to D9602, Q4201 to Q9601, RV4201 to RV9601, RV4202 to RV9602
Changed lines of the file:
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@@
   (symbol (lib_id "power:+12V") (at 133.35 62.23 0)
     (in_bom yes) (on_board yes) (fields_autoplaced)
-    (property "Reference" "#PWR04202" (id 0) (at 133.35 66.04 0)
+    (property "Reference" "#PWR010102" (id 0) (at 133.35 66.04 0)
       (effects (font (size 1.27 1.27)) hide)
     )
@@
   (symbol (lib_id "power:GND") (at 130.81 124.46 0)
     (in_bom yes) (on_board yes) (fields_autoplaced)
-    (property "Reference" "#PWR04201" (id 0) (at 130.81 130.81 0)
+    (property "Reference" "#PWR010101" (id 0) (at 130.81 130.81 0)
       (effects (font (size 1.27 1.27)) hide)
     )
@@
   (symbol (lib_id "power:GND") (at 161.29 76.2 0)
     (in_bom yes) (on_board yes) (fields_autoplaced)
-    (property "Reference" "#PWR04203" (id 0) (at 161.29 82.55 0)
+    (property "Reference" "#PWR010103" (id 0) (at 161.29 82.55 0)
       (effects (font (size 1.27 1.27)) hide)
     )
@@
   (symbol (lib_id "power:GND") (at 176.53 100.33 0)
     (in_bom yes) (on_board yes) (fields_autoplaced)
-    (property "Reference" "#PWR04204" (id 0) (at 176.53 106.68 0)
+    (property "Reference" "#PWR010104" (id 0) (at 176.53 106.68 0)
       (effects (font (size 1.27 1.27)) hide)
     )
@@
   (symbol (lib_id "Device:R") (at 143.51 77.47 0)
     (in_bom yes) (on_board yes) (fields_autoplaced)
-    (property "Reference" "R4201" (id 0) (at 146.05 76.1999 0)
+    (property "Reference" "R9601" (id 0) (at 146.05 76.1999 0)
       (effects (font (size 1.27 1.27)) (justify left))
     )
@@
       (effects (font (size 1.27 1.27)) (justify left))
     )
-    (property "Footprint" "Resistor_THT:R_Axial_DIN0207_L6.3mm_D2.5mm_P2.54mm_Vertical" (id 2) (at 141.732 77.47 90)
+    (property "Footprint" "Resistor_SMD:R_1206_3216Metric_Pad1.30x1.75mm_HandSolder" (id 2) (at 141.732 77.47 90)
       (effects (font (size 1.27 1.27)) hide)
     )
@@
   (symbol (lib_id "Device:R") (at 157.48 69.85 90)
     (in_bom yes) (on_board yes) (fields_autoplaced)
-    (property "Reference" "R4202" (id 0) (at 157.48 63.5 90))
+    (property "Reference" "R9602" (id 0) (at 157.48 63.5 90))
     (property "Value" "47K" (id 1) (at 157.48 66.04 90))
-    (property "Footprint" "Resistor_THT:R_Axial_DIN0207_L6.3mm_D2.5mm_P2.54mm_Vertical" (id 2) (at 157.48 71.628 90)
+    (property "Footprint" "Resistor_SMD:R_1206_3216Metric_Pad1.30x1.75mm_HandSolder" (id 2) (at 157.48 71.628 90)
       (effects (font (size 1.27 1.27)) hide)
     )
@@
   (symbol (lib_id "Device:R") (at 167.64 109.22 0)
     (in_bom yes) (on_board yes) (fields_autoplaced)
-    (property "Reference" "R4203" (id 0) (at 170.18 107.9499 0)
+    (property "Reference" "R9603" (id 0) (at 170.18 107.9499 0)
       (effects (font (size 1.27 1.27)) (justify left))
     )
@@
       (effects (font (size 1.27 1.27)) (justify left))
     )
-    (property "Footprint" "Resistor_THT:R_Axial_DIN0207_L6.3mm_D2.5mm_P2.54mm_Vertical" (id 2) (at 165.862 109.22 90)
+    (property "Footprint" "Resistor_SMD:R_1206_3216Metric_Pad1.30x1.75mm_HandSolder" (id 2) (at 165.862 109.22 90)
       (effects (font (size 1.27 1.27)) hide)
     )
@@
   (symbol (lib_id "Device:D") (at 167.64 116.84 90)
     (in_bom yes) (on_board yes) (fields_autoplaced)
-    (property "Reference" "D4202" (id 0) (at 170.18 115.5699 90)
+    (property "Reference" "D9602" (id 0) (at 170.18 115.5699 90)
       (effects (font (size 1.27 1.27)) (justify right))
     )
@@
   (symbol (lib_id "Device:LED") (at 143.51 104.14 90)
     (in_bom yes) (on_board yes) (fields_autoplaced)
-    (property "Reference" "D4201" (id 0) (at 147.32 103.2508 90)
+    (property "Reference" "D9601" (id 0) (at 147.32 103.2508 90)
       (effects (font (size 1.27 1.27)) (justify right))
     )
@@
   (symbol (lib_id "Device:C_Polarized") (at 118.11 90.17 0)
     (in_bom yes) (on_board yes) (fields_autoplaced)
-    (property "Reference" "C4201" (id 0) (at 121.92 88.8999 0)
+    (property "Reference" "C9601" (id 0) (at 121.92 88.8999 0)
       (effects (font (size 1.27 1.27)) (justify left))
     )
@@
   (symbol (lib_id "Device:R_Potentiometer_Trim") (at 143.51 69.85 90) (mirror x)
     (in_bom yes) (on_board yes) (fields_autoplaced)
-    (property "Reference" "RV4201" (id 0) (at 143.51 63.5 90))
+    (property "Reference" "RV9601" (id 0) (at 143.51 63.5 90))
     (property "Value" "10K TUNE" (id 1) (at 143.51 66.04 90))
     (property "Footprint" "Potentiometer_THT:Potentiometer_Bourns_3386F_Vertical" (id 2) (at 143.51 69.85 0)
@@
   (symbol (lib_id "Device:R_Potentiometer_Trim") (at 167.64 97.79 90) (mirror x)
     (in_bom yes) (on_board yes) (fields_autoplaced)
-    (property "Reference" "RV4202" (id 0) (at 167.64 91.44 90))
+    (property "Reference" "RV9602" (id 0) (at 167.64 91.44 90))
     (property "Value" "100K LVL" (id 1) (at 167.64 93.98 90))
     (property "Footprint" "Potentiometer_THT:Potentiometer_Bourns_3386F_Vertical" (id 2) (at 167.64 97.79 0)
@@
   (symbol (lib_id "Transistor_BJT:2N3904") (at 140.97 90.17 0) (mirror x)
     (in_bom yes) (on_board yes) (fields_autoplaced)
-    (property "Reference" "Q4202" (id 0) (at 146.05 88.8999 0)
+    (property "Reference" "Q9602" (id 0) (at 146.05 88.8999 0)
       (effects (font (size 1.27 1.27)) (justify left))
     )
@@
       (effects (font (size 1.27 1.27)) (justify left))
     )
-    (property "Footprint" "Package_TO_SOT_THT:TO-92_Inline" (id 2) (at 146.05 88.265 0)
+    (property "Footprint" "Package_TO_SOT_SMD:SOT-23" (id 2) (at 146.05 88.265 0)
       (effects (font (size 1.27 1.27) italic) (justify left) hide)
     )
@@
   (symbol (lib_id "Device:Q_NMOS_GDS") (at 128.27 114.3 0) (mirror x)
     (in_bom yes) (on_board yes) (fields_autoplaced)
-    (property "Reference" "Q4201" (id 0) (at 134.62 113.0299 0)
-      (effects (font (size 1.27 1.27)) (justify left))
-    )
+    (property "Reference" "Q9601" (id 0) (at 134.62 113.0299 0)
+      (effects (font (size 1.27 1.27)) (justify left))
+    )
